Commit message: 增加官方测试例程，添加webots接口

File: robot/galileo_mini/urdf/galileo_mini.urdf (robot description, URDF)
Before this commit: robot galileo_mini_description, 18 links, 17 joints
Links:
- removed link world
Joints:
- removed joint RR_foot_joint
- removed joint floating_base_joint
- added joint HR_foot_joint: type fixed, parent HR_knee_link, child HR_foot_link, origin xyz=0.032939 0 -0.26149 rpy=0 0 0, axis 0 0 0
